Commit message: modify files for SO-101

File: config/so_100_arm.ros2_control.xacro (robot description, xacro)
@@ -15,43 +15,43 @@
                 </xacro:unless>
             </hardware>
-            <joint name="Shoulder_Rotation">
+            <joint name="shoulder_pan">
                 <command_interface name="position"/>
                 <state_interface name="position">
-                  <param name="initial_value">${initial_positions['Shoulder_Rotation']}</param>
+                  <param name="initial_value">${initial_positions['shoulder_pan']}</param>
                 </state_interface>
                 <!-- <state_interface name="velocity"/> -->
             </joint>
-            <joint name="Shoulder_Pitch">
+            <joint name="shoulder_lift">
                 <command_interface name="position"/>
                 <state_interface name="position">
-                  <param name="initial_value">${initial_positions['Shoulder_Pitch']}</param>
+                  <param name="initial_value">${initial_positions['shoulder_lift']}</param>
                 </state_interface>
                 <!-- <state_interface name="velocity"/> -->
             </joint>
-            <joint name="Elbow">
+            <joint name="elbow_flex">
                 <command_interface name="position"/>
                 <state_interface name="position">
-                  <param name="initial_value">${initial_positions['Elbow']}</param>
+                  <param name="initial_value">${initial_positions['elbow_flex']}</param>
                 </state_interface>
                 <!-- <state_interface name="velocity"/> -->
             </joint>
-            <joint name="Wrist_Pitch">
+            <joint name="wrist_flex">
                 <command_interface name="position"/>
                 <state_interface name="position">
-                  <param name="initial_value">${initial_positions['Wrist_Pitch']}</param>
+                  <param name="initial_value">${initial_positions['wrist_flex']}</param>
                 </state_interface>
                 <!-- <state_interface name="velocity"/> -->
             </joint>
-            <joint name="Wrist_Roll">
+            <joint name="wrist_roll">
                 <command_interface name="position"/>
                 <state_interface name="position">
-                  <param name="initial_value">${initial_positions['Wrist_Roll']}</param>
+                  <param name="initial_value">${initial_positions['wrist_roll']}</param>
                 </state_interface>
                 <!-- <state_interface name="velocity"/> -->
             </joint>
-            <joint name="Gripper">
+            <joint name="gripper">
                 <command_interface name="position"/>
                 <state_interface name="position">
-                  <param name="initial_value">${initial_positions['Gripper']}</param>
+                  <param name="initial_value">${initial_positions['gripper']}</param>
                 </state_interface>
                 <!-- <state_interface name="velocity"/> -->

File: config/so_100_arm.urdf.xacro (robot description, xacro)
@@ -4,5 +4,5 @@
     <xacro:arg name="use_fake_hardware" default="false"/>
     <!-- Import so_100_arm urdf file -->
-    <xacro:include filename="$(find so_100_arm)/urdf/so_100_arm_5dof_hardware.urdf" />
+    <xacro:include filename="$(find so_100_arm)/urdf/so101_new_calib.urdf" />
     <!-- Import control_xacro -->
     <xacro:include filename="so_100_arm.ros2_control.xacro" />
