Commit message: slight change in urdf

File: urdf/so_100_arm.urdf (robot description, URDF)
Before this commit: robot so_100_arm, 8 links, 7 joints
Links:
- link Fixed_Gripper: geometry collision mesh filename=package://so_100_arm/models/so_100_arm_5dof/meshes/Wrist_Ca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; visual mesh filename=package://so_100_arm/models/so_100_arm_5dof/meshes/Wrist_Ca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
Joints:
- joint Elbow: limit (none) -> lower=-2.8973 upper=2.8973 effort=10.0 velocity=2.175; type continuous -> revolute
- joint Gripper: limit (none) -> lower=-2.8973 upper=2.8973 effort=10.0 velocity=2.175; type continuous -> revolute
- joint Shoulder_Pitch: limit (none) -> lower=-2.8973 upper=2.8973 effort=10.0 velocity=2.175; type continuous -> revolute
- joint Shoulder_Rotation: limit (none) -> lower=-2.8973 upper=2.8973 effort=10.0 velocity=2.175; type continuous -> revolute
- joint Wrist_Pitch: limit (none) -> lower=-2.8973 upper=2.8973 effort=10.0 velocity=2.175; type continuous -> revolute
- joint Wrist_Roll: limit (none) -> lower=-2.8973 upper=2.8973 effort=10.0 velocity=2.175; type continuous -> revolute
